File: PCB/motordriver.brd (EAGLE design)
At the start: 100 x 80 mm, 6 parts

Commit message: work in PCB
Parts:
- added 100K: 55k, myLibrary:0805
- added 100K1: 150k, myLibrary:0805
- added AC1~, AC2~, IN1, IN2, OUT, OUT1: SMDPAD, myLibrary:1.5X7MMPAD
- added B1: RECTIFIER-GBU4, rectifier:GBU4
- added BC47HFE=10000: MMBTA14LT1, transistor-npn:SOT23-BEC
- added BC846, BC846$: (no value), semicon-smd-ipc:SOT23
- added C1: 10000uF/25V, rcl:E7,5-18
- added C2: 0.1uF, rcl:C1206
- added C3: 0.330uF, rcl:C1206
- added C4, C6: 47nF, rcl:C1206K
- added C5: 1uF, rcl:C1206K
- added C7: 100nF, rcl:C1206
- added FUSE: 100mA(hold), myLibrary:0805
- added GREEN_LED, RED_LED: (no value), led:CHIPLED_0805
- added IC1: 7818TV, linear:TO220V
- added JMP1, JMP2, JMP3: 0R-JUMPA, jump-0r-smd:A0R-JMP
- added R5, R6: 420 Ohm, myLibrary:0805
- added R7: 68k 1%, resistor:R0805
- added R8: 10k, resistor:R0805
- added R9: 12k, myLibrary:0805
- added U$3: POWER_LED, myLibrary:OSRAMLED
- R1: value (none) -> 320
- R2: value (none) -> 10k
- R3: value (none) -> 132
- R4: value (none) -> 7 2W; device eagle-ltspice:R0805 -> resistor:R1210
- moved U$1 74.5 mm to (86.7, 62.0)
- moved R3 48.5 mm to (72.6, 17.5), turned to 270 degrees
- moved R1 44.5 mm to (67.8, 17.6), turned to 90 degrees
- moved U$2 43.4 mm to (45.5, 44.9)
- moved R2 32.5 mm to (29.4, 46.9), turned to 270 degrees
- moved R4 8.02 mm to (31.4, 4.75), turned to 270 degrees
Connections:
- net N$1 renamed GND1
- removed net CPH: U$2.22
- removed net CPL: U$2.23
- removed net VCP: U$2.21
- removed net VM_A: U$2.13
- removed net VM_B: U$2.20
- new net +12V: B1.+, C1.+, C3.1, C6.1, IC1.1, U$2.13, U$2.20
- new net +5V: C2.1, FUSE.P$1, IC1.3, R1.P$1, R3.P$1, R4.1
- new net 120MA: BC47HFE=10000.C, U$3.C1, U$3.C2
- new net 22MA: BC846$.3, RED_LED.C
- new net 3.3V: R2.P$2, R8.1, U$1.P$23
- new net 5MA: BC846.3, GREEN_LED.C
- new net BUTTON: C7.1, IN1.P$1, R2.P$1
- new net N$1: AC1~.P$1, B1.AC1
- new net N$10: R7.2, U$2.4
- new net N$11: C6.2, U$2.21
- new net N$12: OUT1.P$1, U$2.14, U$2.15
- new net N$13: OUT.P$1, U$2.18, U$2.19
- new net N$14: R3.P$2, RED_LED.A
- new net N$15: GREEN_LED.A, R1.P$2
- new net N$18: BC846$.1, R9.P$2
- new net N$19: R9.P$1
- new net N$2: AC2~.P$1, B1.AC2
- new net N$20: 100K.P$2, BC846.1
- new net N$21: 100K.P$1
- new net N$23: R4.2, U$3.A1, U$3.A2
- new net N$24: 100K1.P$2, BC47HFE=10000.B
- new net N$25: 100K1.P$1
- new net N$26: FUSE.P$2, U$1.P$17
- new net N$3: C4.1, U$2.22
- new net N$4: C4.2, U$2.23
- new net N$5: JMP2.2, U$2.6
- new net N$6: R6.P$2, U$2.12
- new net N$7: R5.P$2, U$2.10
- new net N$8: JMP1.2, U$2.5
- new net N$9: JMP3.2, U$2.3
- new net TOARM: R8.2, U$2.2
- net DVDD: now also C5.2, JMP1.1, JMP2.1, JMP3.1
- net GND: now also B1.-, BC47HFE=10000.E, BC846$.2, BC846.2, C1.-, C2.2, C3.2, C5.1, C7.2, IC1.2, IN2.P$1, JMP1.3, JMP2.3, JMP3.3, R5.P$1, R6.P$1, R7.1, U$2.16, U$2.17

Commit message: work in board
Parts:
- removed 100K: 55k, myLibrary:0805
- added AC1~1, AC2~1, IN3, IN4, OUT2, OUT3: SMDPAD, myLibrary:1.5X7MMPAD
- added C8, C9: 100nF, rcl:C0805
- added R10: 55k, myLibrary:0805
- C6: value 47nF -> 1uF
- moved R2 34.1 mm to (60.4, 61.2), turned to 0 degrees
- moved BC846 19.3 mm to (85.5, 5.15), turned to 270 degrees
- moved R1 17.5 mm to (85.2, 18.9), turned to 0 degrees
- moved C7 14.4 mm to (60.9, 66.0)
- moved R5 13.8 mm to (39.8, 43.5)
- moved R3 12.9 mm to (85.2, 14.8), turned to 0 degrees
- moved BC846$ 10.6 mm to (85.5, 9.65), turned to 270 degrees
- moved R9 8.85 mm to (78.5, 11.5), turned to 270 degrees
- moved R6 8.55 mm to (40.3, 40.0), turned to 90 degrees
- moved 100K1 8.45 mm to (62.0, 11.3), turned to 270 degrees
- moved JMP2 7.68 mm to (30.2, 57.5)
- moved BC47HFE=10000 5.94 mm to (63.2, 6.35), turned to 270 degrees
- moved C6 4.76 mm to (51.9, 47.4)
- moved JMP3 4.11 mm to (40.9, 57.5)
- moved JMP1 3.96 mm to (35.6, 57.5)
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Connections:
- removed net BUTTON: C7.1, IN1.P$1, R2.P$1
- removed net GND1: U$1.P$21
- removed net N$19: R9.P$1
- removed net N$21: 100K.P$1
- removed net N$25: 100K1.P$1
- removed net N$6: R6.P$2, U$2.12
- removed net N$7: R5.P$2, U$2.10
- new net PA0: R6.P$2, U$1.P$36, U$2.12
- new net PA1: R5.P$2, U$1.P$35, U$2.10
- new net PA15: C7.1, IN1.P$1, IN3.P$1, R2.P$1, U$1.P$10
- new net PB0: U$1.P$28
- new net PB11: U$1.P$25, U$2.11
- new net PB12: R9.P$1, U$1.P$1
- new net PB13: R10.P$1, U$1.P$2
- new net PB14: 100K1.P$1, U$1.P$3
- new net PB3: U$1.P$11
- new net PB4: U$1.P$12, U$2.9
- new net PB8: U$1.P$16, U$2.8
- new net PB9: U$1.P$17, U$2.7
- net +12V: now also C8.2, C9.1
- net GND: now also C8.1, C9.2, IN4.P$1, U$1.P$19, U$1.P$21, U$1.P$22
- net N$1: now also AC1~1.P$1
- net N$12: now also OUT3.P$1
- net N$13: now also OUT2.P$1
- net N$2: now also AC2~1.P$1
- net N$20: now also R10.P$2; no longer 100K.P$2
- net N$26: now also U$1.P$18; no longer U$1.P$17
Routing:
- net GND: track 0.00 -> 221.3 mm, vias 0 -> 2
- net +12V: track 0.00 -> 94.2 mm
- net PB14: track 0.00 -> 82.4 mm
- net PB13: track 0.00 -> 79.0 mm
- net PB12: track 0.00 -> 75.9 mm
- net +5V: track 0.00 -> 51.8 mm
- net N$1: track 0.00 -> 51.6 mm, vias 0 -> 1
- net N$2: track 0.00 -> 51.0 mm, vias 0 -> 1
- net N$8: track 0.00 -> 34.8 mm
- net N$5: track 0.00 -> 33.9 mm
- net N$9: track 0.00 -> 29.6 mm
- net DVDD: track 0.00 -> 27.4 mm
- net PA15: track 0.00 -> 18.7 mm, vias 0 -> 1
- net 5MA: track 0.00 -> 18.1 mm
- net N$23: track 0.00 -> 17.6 mm
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
Commit message: more work in board
Parts:
- moved C8 5.71 mm to (53.8, 54.8)
- moved C4 5.68 mm to (51.2, 50.6)
- moved C9 3.43 mm to (50.3, 38.9), turned to 270 degrees
- moved C6 2.85 mm to (54.8, 47.3)
Routing:
- net +5V: track 51.8 -> 109.5 mm
- net +12V: track 94.2 -> 147.9 mm, vias 0 -> 3
- net N$12: track 0.21 -> 45.3 mm, vias 0 -> 2
- net N$13: track 0.07 -> 40.2 mm, vias 0 -> 2
- net N$11: track 0.12 -> 7.65 mm
- net N$4: track 0.00 -> 6.10 mm
- net N$3: track 0.12 -> 3.85 mm

Commit message: more work in board
Connections:
- net 3.3V: now also U$1.P$20
Routing:
- net 3.3V: track 0.18 -> 97.6 mm, vias 0 -> 2
- net PB11: track 8.32 -> 94.0 mm, vias 0 -> 2
- net PA1: track 3.12 -> 85.2 mm, vias 0 -> 1
- net PA0: track 2.64 -> 60.1 mm, vias 0 -> 1
- net PB4: track 9.73 -> 65.0 mm, vias 0 -> 1
- net PB8: track 10.6 -> 61.8 mm
- net PB9: track 11.5 -> 61.8 mm
- net GND: track 221.3 -> 252.9 mm, vias 2 -> 17
- net PA15: track 18.5 -> 46.5 mm, vias 1 -> 2
- net +5V: track 109.5 -> 123.4 mm, vias 0 -> 2
- net N$26: track 0.05 -> 8.95 mm
- net +12V: track 147.9 -> 153.1 mm
- net N$12: track 45.3 -> 50.0 mm, vias 2 -> 3
- net N$13: track 40.2 -> 44.8 mm, vias 2 -> 3
- added copper zone on layer 16, net GND

Commit message: more work in board
Connections:
- net GND: no longer U$2.PS$1, U$2.PS$10, U$2.PS$11, U$2.PS$12, U$2.PS$13, U$2.PS$14, U$2.PS$15, U$2.PS$16, U$2.PS$17, U$2.PS$18, U$2.PS$2, U$2.PS$3, U$2.PS$4, U$2.PS$5, U$2.PS$6, U$2.PS$7, U$2.PS$8, U$2.PS$9
Routing:
- net +12V: track 153.1 -> 146.0 mm
- net GND: track 252.9 -> 248.6 mm, vias 17 -> 25
